Commit message: r2000修改

File: urdf/whillcar.urdf (robot description, URDF)
Before this commit: robot whillcar, 6 links, 5 joints
Joints:
- joint left_wheel_joint: origin xyz=0 ${-wheel_separation/2} ${wheel_radius} rpy=${pi/2} 0 0 -> xyz=0 ${wheel_separation/2} ${wheel_radius} rpy=${pi/2} 0 0
- joint right_wheel_joint: origin xyz=0 ${wheel_separation/2} ${wheel_radius} rpy=${pi/2} 0 0 -> xyz=0 ${-wheel_separation/2} ${wheel_radius} rpy=${pi/2} 0 0

Commit message: 一些调整

File: urdf/whillcar.urdf (robot description, URDF)
Before this commit: robot whillcar, 6 links, 5 joints
Joints:
- joint imu_joint: origin xyz=${imu_x} ${imu_y} ${imu_z} rpy=0 0 0 -> xyz=${imu_x} ${imu_y} ${imu_z} rpy=0 0 ${pi}
- joint laser_joint: origin xyz=${laser_x} ${laser_y} ${laser_z} rpy=0 0 0 -> xyz=${laser_x} ${laser_y} ${laser_z} rpy=0 0 ${-pi/2}

Commit message: 双雷达版本！

File: urdf/whillcar.urdf (robot description, URDF)
Before this commit: robot whillcar, 6 links, 5 joints
Links:
- added link laser_left_frame, mass ${laser_mass}; collision cylinder length=${laser_size} radius=${laser_size/2}; visual cylinder length=${laser_size} radius=${laser_size/2}
- added link laser_right_frame, mass ${laser_mass}; collision cylinder length=${laser_size} radius=${laser_size/2}; visual cylinder length=${laser_size} radius=${laser_size/2}
Joints:
- added joint laser_left_joint: type fixed, parent base_link, child laser_left_frame, origin xyz=${laser_dual_x} ${laser_dual_y} ${laser_z} rpy=0 0 ${laser_left_yaw}
- added joint laser_right_joint: type fixed, parent base_link, child laser_right_frame, origin xyz=${laser_dual_x} ${-laser_dual_y} ${laser_z} rpy=0 0 ${laser_right_yaw}

Commit message: 111

File: urdf/whillcar.urdf (robot description, URDF)
Before this commit: robot whillcar, 8 links, 7 joints
Links:
- removed link laser_frame
Joints:
- removed joint laser_joint
